File: 0025_Sound_Module_MAX4466.kicad_sch (KiCad schematic)
At the start: 15 parts, among them U1 MAX4466EXK

Commit message: Add files via upload
Parts:
- added D1: LED, LED_SMD:LED_0805_2012Metric, symbol Device:LED
- added R7: R, Resistor_SMD:R_0805_2012Metric, symbol Device:R
- added U2: ~, Moduler_:pin_header, symbol moduler_pin:air
- C1, C2, C3, C4: footprint (none) -> Capacitor_SMD:C_0805_2012Metric
- FB1, FB2: footprint (none) -> Inductor_SMD:L_0805_2012Metric
- MK1: footprint MIC_CMA-4544PF-W -> CMA4544:MIC_CMA-4544PF-W
- R1, R2, R3, R4, R5, R6: footprint (none) -> Resistor_SMD:R_0805_2012Metric
- RV1: footprint (none) -> meminle:3362P_1
- U1: footprint SOT65P210X110-5N -> meminle:SOT65P210X110-5N
Connections:
- net GND: now also D1.1 (K), U2.9; no longer C1.1, C3.1, FB2.2, MK1.2, R2.2, U1.2 (GND)
- net OUT: now reaches C2.1, RV1.1, RV1.2, U1.4 (OUT)
- net OUT: now also U2.12
- net VCC renamed +3.3VA
- net +3.3VA: no longer FB1.1
- new net: D1.2 (A), R7.2
- new net +3V3: FB1.1, R7.1, U2.8
- new net GND1: C1.1, C3.1, FB2.2, MK1.2, R2.2, U1.2 (GND)
- no-connect marks 0 -> 15
Other:
- note added: "AIR PIN"
- note added: "SENSOR"
- moved on the sheet: C1, C2, C3, C4, FB1, FB2, MK1, R1, R2, R3, R4, R5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
